File: Hardware/PUTM_EV_Frontbox_2023/apps1.kicad_sch (KiCad schematic)
At the start: 12 parts, among them U13 TLV9152IDDFR

Commit message: Written firmware
Parts:
- R30: value 10k -> 4k
- R35, R37: value 60k3 -> 40k
Other:
- note added: "0.34V - 0.79V"
- note added: "APPS2 2.34V to 2.79V"
- note added: "Amplification by 4"
- note removed: "APPS1 2.56V to 2.94V"
- note removed: "Amplification by 6"
Changed lines of the file:
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@@
     )
   )
-  (text "Amplification by 6" (at 115.57 95.25 0)
+  (text "0.34V - 0.79V" (at 92.71 88.265 0)
     (effects (font (size 1.27 1.27)) (justify left bottom))
   )
+  (text "Amplification by 4" (at 113.665 95.25 0)
+    (effects (font (size 1.27 1.27)) (justify left bottom))
+  )
+  (text "APPS2\n2.34V to 2.79V" (at 19.05 91.44 0)
+    (effects (font (size 1.27 1.27)) (justify left bottom))
+  )
   (text "Sallen Key LPF f_{c} = 300 Hz" (at 61.595 118.745 0)
-    (effects (font (size 1.27 1.27)) (justify left bottom))
-  )
-  (text "APPS1\n2.56V to 2.94V\n" (at 31.115 90.17 0)
     (effects (font (size 1.27 1.27)) (justify left bottom))
   )
@@
       (effects (font (size 1.27 1.27)))
     )
-    (property "Value" "60k3" (at 139.065 116.84 90)
+    (property "Value" "40k" (at 139.065 116.84 90)
       (effects (font (size 1.27 1.27)))
     )
@@
       (effects (font (size 1.27 1.27)) (justify left))
     )
-    (property "Value" "10k" (at 27.94 101.6 0)
+    (property "Value" "4k" (at 27.94 101.6 0)
       (effects (font (size 1.27 1.27)) (justify left))
     )
@@
   (symbol (lib_id "Device:R_Small") (at 111.125 108.585 0) (mirror y) (unit 1)
     (in_bom yes) (on_board yes) (dnp no)
-    (property "Reference" "R35" (at 109.22 107.95 0)
-      (effects (font (size 1.27 1.27)) (justify left))
-    )
-    (property "Value" "60k3" (at 109.22 110.49 0)
-      (effects (font (size 1.27 1.27)) (justify left))
-    )
+    (property "Reference" "R35" (at 109.855 107.95 0)
+      (effects (font (size 1.27 1.27)) (justify left))
+    )
+    (property "Value" "40k" (at 109.855 109.855 0)
+      (effects (font (size 1.27 1.27)) (justify left))
+    )
