File: Hardware/PUTM_EV_Frontbox_2023/PUTM_EV_Frontbox_2023.kicad_pcb (KiCad board)
At the start: 2 copper layers, 60 x 40 mm, 4 parts

Commit message: Grouped components
Parts:
- removed REF** (x4): MountingHole_3.5mm_Pad_Via, MountingHole:MountingHole_3.5mm_Pad_Via
- added C1: 100nF, Capacitor_SMD:C_0402_1005Metric_Pad0.74x0.62mm_HandSolder, F.Cu at (116.0, 68.2)
- added C10: 100nF, Capacitor_SMD:C_0402_1005Metric_Pad0.74x0.62mm_HandSolder, F.Cu at (125.1, 99.2)
- added C11: 100nF, Capacitor_SMD:C_0402_1005Metric_Pad0.74x0.62mm_HandSolder, F.Cu at (130.2, 87.0)
- added C12: 1uF, Capacitor_SMD:C_0402_1005Metric_Pad0.74x0.62mm_HandSolder, F.Cu at (56.3, 180.2)
- added C13: 100nF, Capacitor_SMD:C_0402_1005Metric_Pad0.74x0.62mm_HandSolder, F.Cu at (127.2, 89.6)
- added C14: 1uF, Capacitor_SMD:C_0402_1005Metric_Pad0.74x0.62mm_HandSolder, F.Cu at (67.0, 175.7)
- added C15: 1uF, Capacitor_SMD:C_0402_1005Metric_Pad0.74x0.62mm_HandSolder, F.Cu at (80.0, 165.8)
- added C16: 1uF, Capacitor_SMD:C_0402_1005Metric_Pad0.74x0.62mm_HandSolder, F.Cu at (88.1, 157.7)
- added C17: 10nF, Capacitor_SMD:C_0402_1005Metric_Pad0.74x0.62mm_HandSolder, F.Cu at (164.3, 158.2)
- added C18: 1uF, Capacitor_SMD:C_0402_1005Metric_Pad0.74x0.62mm_HandSolder, F.Cu at (47.4, 140.1)
- added C19: 100nF, Capacitor_SMD:C_0402_1005Metric_Pad0.74x0.62mm_HandSolder, F.Cu at (156.1, 103.8)
- added C20: 100nF, Capacitor_SMD:C_0402_1005Metric_Pad0.74x0.62mm_HandSolder, F.Cu at (149.5, 100.3)
- added C23: 10pF, Capacitor_SMD:C_0402_1005Metric_Pad0.74x0.62mm_HandSolder, F.Cu at (118.5, 90.3)
- added C24: 10pF, Capacitor_SMD:C_0402_1005Metric_Pad0.74x0.62mm_HandSolder, F.Cu at (118.3, 99.2)
- added C25: 100n, Capacitor_SMD:C_0402_1005Metric_Pad0.74x0.62mm_HandSolder, F.Cu at (149.8, 18.9)
- added C26: 47n 1%, Capacitor_SMD:C_0402_1005Metric_Pad0.74x0.62mm_HandSolder, F.Cu at (122.3, 192.7)
- added C27: 47n 1%, Capacitor_SMD:C_0402_1005Metric_Pad0.74x0.62mm_HandSolder, F.Cu at (116.1, 187.6)
- added C28: 100n, Capacitor_SMD:C_0402_1005Metric_Pad0.74x0.62mm_HandSolder, F.Cu at (108.3, 180.0)
- added C29: 100n, Capacitor_SMD:C_0402_1005Metric_Pad0.74x0.62mm_HandSolder, F.Cu at (75.7, 23.4)
- added C3: 100nF, Capacitor_SMD:C_0402_1005Metric_Pad0.74x0.62mm_HandSolder, F.Cu at (131.3, 80.1)
- added C33: 47n 1%, Capacitor_SMD:C_0402_1005Metric_Pad0.74x0.62mm_HandSolder, F.Cu at (150.3, 182.8)
- added C34: 47n 1%, Capacitor_SMD:C_0402_1005Metric_Pad0.74x0.62mm_HandSolder, F.Cu at (142.9, 179.8)
- added C35: 100n, Capacitor_SMD:C_0402_1005Metric_Pad0.74x0.62mm_HandSolder, F.Cu at (162.5, 179.6)
- added C36: 1uF, Capacitor_SMD:C_0402_1005Metric_Pad0.74x0.62mm_HandSolder, F.Cu at (87.6, 162.2)
- added C37: 1uF, Capacitor_SMD:C_0402_1005Metric_Pad0.74x0.62mm_HandSolder, F.Cu at (72.8, 161.1)
- added C38: 1uF, Capacitor_SMD:C_0402_1005Metric_Pad0.74x0.62mm_HandSolder, F.Cu at (65.2, 139.4)
- added C39: 10uF, Capacitor_SMD:CP_Elec_4x5.7, F.Cu at (135.6, 121.1)
- added C4: 100nF, Capacitor_SMD:C_0402_1005Metric_Pad0.74x0.62mm_HandSolder, F.Cu at (136.2, 80.6)
- added C40: 100nF, Capacitor_SMD:C_0402_1005Metric_Pad0.74x0.62mm_HandSolder, F.Cu at (112.2, 134.1)
- added C41: 220nF, Capacitor_SMD:C_0402_1005Metric_Pad0.74x0.62mm_HandSolder, F.Cu at (203.6, 161.0)
- added C43: 1uF, Capacitor_SMD:C_0402_1005Metric_Pad0.74x0.62mm_HandSolder, F.Cu at (198.6, 162.3)
- added C44: 220nF, Capacitor_SMD:C_0402_1005Metric_Pad0.74x0.62mm_HandSolder, F.Cu at (214.4, 159.2)
- added C45: 4u7F, Capacitor_SMD:CP_Elec_4x5.7, F.Cu at (203.1, 142.7)
- added C46: 100nF, Capacitor_SMD:C_0402_1005Metric_Pad0.74x0.62mm_HandSolder, F.Cu at (191.6, 155.1)
- added C47: 10uF, Capacitor_SMD:CP_Elec_4x5.7, F.Cu at (204.4, 150.3)
- added C5: 100nF, Capacitor_SMD:C_0402_1005Metric_Pad0.74x0.62mm_HandSolder, F.Cu at (112.2, 132.1)
- added C6: 1uF, Capacitor_SMD:C_0402_1005Metric_Pad0.74x0.62mm_HandSolder, F.Cu at (126.1, 113.5)
- added C7: 100nF, Capacitor_SMD:C_0402_1005Metric_Pad0.74x0.62mm_HandSolder, F.Cu at (127.7, 108.4)
- added C8: 100nF, Capacitor_SMD:C_0402_1005Metric_Pad0.74x0.62mm_HandSolder, F.Cu at (137.3, 104.8)
- added C9: 100nF, Capacitor_SMD:C_0402_1005Metric_Pad0.74x0.62mm_HandSolder, F.Cu at (142.4, 92.1)
- added D1: LED, LED_SMD:LED_0201_0603Metric, F.Cu at (194.3, 25.1)
- added D2: LED, LED_SMD:LED_0201_0603Metric, F.Cu at (185.2, 27.6)
- added D3: LED, LED_SMD:LED_0201_0603Metric, F.Cu at (185.2, 32.2)
- added D4: LED, LED_SMD:LED_0201_0603Metric, F.Cu at (185.0, 35.7)
- added D5: LED, LED_SMD:LED_0201_0603Metric, F.Cu at (196.7, 37.8)
- added D6: SD24_SOD323, Diode_SMD:D_SOD-323_HandSoldering, F.Cu at (188.4, 159.2)
- added F1: 1A, Fuse:Fuse_1812_4532Metric_Pad1.30x3.40mm_HandSolder, F.Cu at (190.6, 141.4)
- added F2: 300mA, Fuse:Fuse_0603_1608Metric_Pad1.05x0.95mm_HandSolder, F.Cu at (60.1, 179.5)
- added F3: 300mA, Fuse:Fuse_0603_1608Metric_Pad1.05x0.95mm_HandSolder, F.Cu at (52.5, 138.9)
- added F4: 1.5A, Fuse:Fuse_1812_4532Metric_Pad1.30x3.40mm_HandSolder, F.Cu at (175.7, 90.6)
- added FB1: 1000Ω@100MHz, Inductor_SMD:L_0603_1608Metric, F.Cu at (136.9, 107.4)
- added FB2: 60R@100MHz, Inductor_SMD:L_0603_1608Metric, F.Cu at (152.3, 103.9)
- added FB4: 60R@100MHz, Inductor_SMD:L_0603_1608Metric, F.Cu at (109.6, 127.3)
- added FB5: 60R@100MHz, Inductor_SMD:L_0603_1608Metric, F.Cu at (109.6, 129.8)
- added FB6: 60R@100MHz, Inductor_SMD:L_0603_1608Metric, F.Cu at (133.4, 77.5)
- added H1: M3, MountingHole:MountingHole_2mm, F.Cu at (30.2, 155.2)
- added H10: M3, MountingHole:MountingHole_2mm, F.Cu at (35.7, 177.4)
- added H2: M3, MountingHole:MountingHole_2mm, F.Cu at (30.2, 160.7)
- added H3: M3, MountingHole:MountingHole_2mm, F.Cu at (30.2, 166.3)
- added H4: M3, MountingHole:MountingHole_2mm, F.Cu at (30.2, 171.8)
- added H5: M3, MountingHole:MountingHole_2mm, F.Cu at (30.2, 177.4)
- added H6: M3, MountingHole:MountingHole_2mm, F.Cu at (35.7, 155.2)
- added H7: M3, MountingHole:MountingHole_2mm, F.Cu at (35.7, 160.7)
- added H8: M3, MountingHole:MountingHole_2mm, F.Cu at (35.7, 166.3)
- added H9: M3, MountingHole:MountingHole_2mm, F.Cu at (35.7, 171.8)
- added IC1: ELVH-MF12D-HRRJ-C-N3A4, Frontbox:ELVH005DHRRJINAA4, F.Cu at (101.1, 131.0)
- added IC2: ELVH-MF12D-HRRJ-C-N3A4, Frontbox:ELVHL10DHRRDCN2A4, F.Cu at (94.0, 112.4)
- added J1: Złącze TE, Frontbox:Autosport, F.Cu at (267.6, 94.2)
- added J2: Conn_01x04, Connector_PinHeader_1.00mm:PinHeader_1x05_P1.00mm_Vertical, F.Cu at (102.3, 52.0)
- added J3: Conn_02x14_Counter_Clockwise, Connector_PinHeader_2.54mm:PinHeader_2x14_P2.54mm_Horizontal, F.Cu at (245.0, 114.0)
- added J4: USB_C_Receptacle, Connector_USB:USB_C_Receptacle_G-Switch_GT-USB-7010ASV, F.Cu at (131.2, 55.0)
- added J5: Conn_02x14_Counter_Clockwise, Connector_PinSocket_2.54mm:PinSocket_2x14_P2.54mm_Horizontal, F.Cu at (182.0, 113.5)
- added K1: UMS05-1A80-75D, Relay_THT:Relay_StandexMeder_UMS, F.Cu at (180.5, 128.7)
- added L1: 2u2H, Inductor_SMD:L_Abracon_ASPI-4030S, F.Cu at (192.2, 149.5)
- added Q1: NX7002AK, Package_TO_SOT_SMD:SOT-23, F.Cu at (171.5, 129.2)
- added R1: 100R, Resistor_SMD:R_0402_1005Metric, F.Cu at (197.0, 25.1)
- added R10: 10k, Resistor_SMD:R_0402_1005Metric, F.Cu at (167.8, 130.2)
- added R11: 2k, Resistor_SMD:R_0402_1005Metric, F.Cu at (41.6, 101.8)
- added R12: 2k, Resistor_SMD:R_0402_1005Metric, F.Cu at (41.6, 104.6)
- added R13: 2k, Resistor_SMD:R_0402_1005Metric, F.Cu at (41.8, 107.1)
- added R14: 2k, Resistor_SMD:R_0402_1005Metric, F.Cu at (41.8, 109.4)
- added R15: 2k, Resistor_SMD:R_0402_1005Metric, F.Cu at (39.3, 75.9)
- added R16: 2k, Resistor_SMD:R_0402_1005Metric, F.Cu at (39.3, 78.5)
- added R17: 5k, Resistor_SMD:R_0402_1005Metric, F.Cu at (136.1, 33.2)
- added R18: 5k, Resistor_SMD:R_0402_1005Metric, F.Cu at (156.1, 26.6)
- added R19: 200R, Resistor_SMD:R_0402_1005Metric, F.Cu at (49.5, 182.7)
- added R2: 100R, Resistor_SMD:R_0402_1005Metric, F.Cu at (187.9, 27.6)
- added R20: 10k, Resistor_SMD:R_0402_1005Metric, F.Cu at (118.3, 19.2)
- added R21: 10k, Resistor_SMD:R_0402_1005Metric, F.Cu at (118.3, 22.3)
- added R22: 3k, Resistor_SMD:R_0402_1005Metric, F.Cu at (122.1, 21.0)
- added R23: 3k, Resistor_SMD:R_0402_1005Metric, F.Cu at (135.3, 22.0)
- added R24: 12k, Resistor_SMD:R_0402_1005Metric, F.Cu at (134.0, 29.4)
- added R25: 12k, Resistor_SMD:R_0402_1005Metric, F.Cu at (138.4, 24.6)
- added R26: 3k, Resistor_SMD:R_0402_1005Metric, F.Cu at (138.6, 22.0)
- added R27: 3k, Resistor_SMD:R_0402_1005Metric, F.Cu at (149.8, 22.5)
- added R28: 12k, Resistor_SMD:R_0402_1005Metric, F.Cu at (138.9, 20.0)
- added R29: 12k, Resistor_SMD:R_0402_1005Metric, F.Cu at (153.6, 21.3)
- added R3: 100R, Resistor_SMD:R_0402_1005Metric, F.Cu at (188.4, 32.2)
- added R30: R_Small, Resistor_SMD:R_0402_1005Metric, F.Cu at (94.9, 181.8)
- added R31: R_Small, Resistor_SMD:R_0402_1005Metric, F.Cu at (94.9, 185.3)
- added R32: 10k 1%, Resistor_SMD:R_0402_1005Metric, F.Cu at (111.3, 192.2)
- added R33: 10k 1%, Resistor_SMD:R_0402_1005Metric, F.Cu at (115.2, 192.2)
- added R34: R_Small, Resistor_SMD:R_0402_1005Metric, F.Cu at (125.6, 180.0)
- added R35: R_Small, Resistor_SMD:R_0402_1005Metric, F.Cu at (129.9, 182.0)
- added R36: R_Small, Resistor_SMD:R_0402_1005Metric, F.Cu at (102.7, 190.2)
- added R37: R_Small, Resistor_SMD:R_0402_1005Metric, F.Cu at (106.3, 190.2)
- added R38: R_Small, Resistor_SMD:R_0402_1005Metric, F.Cu at (58.2, 21.4)
- added R39: R_Small, Resistor_SMD:R_0402_1005Metric, F.Cu at (58.2, 28.0)
- added R4: 100R, Resistor_SMD:R_0402_1005Metric, F.Cu at (188.4, 35.7)
- added R40: R_Small, Resistor_SMD:R_0402_1005Metric, F.Cu at (68.2, 36.2)
- added R41: R_Small, Resistor_SMD:R_0402_1005Metric, F.Cu at (76.1, 36.1)
- added R42: R_Small, Resistor_SMD:R_0402_1005Metric, F.Cu at (64.6, 35.6)
- added R43: R_Small, Resistor_SMD:R_0402_1005Metric, F.Cu at (78.7, 31.7)
- added R44: R_Small, Resistor_SMD:R_0402_1005Metric, F.Cu at (68.8, 27.9)
- added R45: R_Small, Resistor_SMD:R_0402_1005Metric, F.Cu at (83.0, 28.6)
- added R46: R_Small, Resistor_SMD:R_0402_1005Metric, F.Cu at (71.5, 37.6)
- added R47: R_Small, Resistor_SMD:R_0402_1005Metric, F.Cu at (74.7, 40.5)
- added R48: 10k, Resistor_SMD:R_0402_1005Metric, F.Cu at (54.5, 80.4)
- added R49: 2k, Resistor_SMD:R_0402_1005Metric, F.Cu at (39.2, 83.6)
- added R5: 100R, Resistor_SMD:R_0402_1005Metric, F.Cu at (199.1, 37.8)
- added R50: 10k, Resistor_SMD:R_0402_1005Metric, F.Cu at (54.4, 83.0)
- added R67: R_Small, Resistor_SMD:R_0402_1005Metric, F.Cu at (153.1, 188.4)
- added R68: R_Small, Resistor_SMD:R_0402_1005Metric, F.Cu at (153.1, 191.7)
- added R69: 10k 1%, Resistor_SMD:R_0402_1005Metric, F.Cu at (140.4, 181.5)
- added R70: 10k 1%, Resistor_SMD:R_0402_1005Metric, F.Cu at (145.5, 181.5)
- added R71: R_Small, Resistor_SMD:R_0402_1005Metric, F.Cu at (159.7, 188.9)
- added R72: R_Small, Resistor_SMD:R_0402_1005Metric, F.Cu at (162.5, 189.7)
- added R73: R_Small, Resistor_SMD:R_0402_1005Metric, F.Cu at (166.0, 185.8)
- added R74: R_Small, Resistor_SMD:R_0402_1005Metric, F.Cu at (167.3, 182.0)
- added R75: 220R, Resistor_SMD:R_0402_1005Metric, F.Cu at (72.1, 179.5)
- added R76: 10k, Resistor_SMD:R_0402_1005Metric, F.Cu at (131.7, 20.5)
- added R77: 10k, Resistor_SMD:R_0402_1005Metric, F.Cu at (131.7, 23.5)
- added R79: 10k, Resistor_SMD:R_0402_1005Metric, F.Cu at (55.7, 101.4)
- added R80: 10k, Resistor_SMD:R_0402_1005Metric, F.Cu at (55.7, 104.1)
- added R81: 10k, Resistor_SMD:R_0402_1005Metric, F.Cu at (55.7, 106.6)
- added R82: 10k, Resistor_SMD:R_0402_1005Metric, F.Cu at (55.7, 109.1)
- added R83: 10k, Resistor_SMD:R_0402_1005Metric, F.Cu at (54.4, 75.5)
- added R84: 10k, Resistor_SMD:R_0402_1005Metric, F.Cu at (54.4, 78.0)
- added R85: 4k7, Resistor_SMD:R_0402_1005Metric, F.Cu at (109.1, 132.1)
- added R86: 4k7, Resistor_SMD:R_0402_1005Metric, F.Cu at (109.1, 134.1)
- added R87: 100k, Resistor_SMD:R_0402_1005Metric, F.Cu at (49.5, 186.7)
- added R88: 16k7, Resistor_SMD:R_0402_1005Metric, F.Cu at (49.5, 188.7)
- added R89: 0R, Resistor_SMD:R_0402_1005Metric, F.Cu at (195.8, 155.1)
- added R9: 200R, Resistor_SMD:R_0402_1005Metric, F.Cu at (164.3, 128.2)
- added R93: 2k, Resistor_SMD:R_0402_1005Metric, F.Cu at (39.3, 80.9)
- added SW1: Reset switch, Button_Switch_SMD:SW_MEC_5GSH9, F.Cu at (113.5, 59.6)
- added TP1: TestPoint, TestPoint:TestPoint_Pad_1.0x1.0mm, F.Cu at (146.5, 90.6)
- added TP2: TestPoint, TestPoint:TestPoint_Pad_1.0x1.0mm, F.Cu at (146.5, 98.2)
- added TP4: TestPoint_2Pole, TestPoint:TestPoint_2Pads_Pitch2.54mm_Drill0.8mm, F.Cu at (109.5, 124.4)
- added U1: STM32G473RCTx, Package_QFP:LQFP-64_10x10mm_P0.5mm, F.Cu at (133.8, 95.7)
- added U10: TLP291-4, Package_SO:SOIC-16_4.55x10.3mm_P1.27mm, F.Cu at (48.7, 106.3)
- added U11: TLP291-4, Package_SO:SOIC-16_4.55x10.3mm_P1.27mm, F.Cu at (46.4, 80.4)
- added U12: TLV9152IDDFR, Package_TO_SOT_SMD:TSOT-23-8_HandSoldering, F.Cu at (144.1, 21.0)
- added U13: TLV9152IDDFR, Package_TO_SOT_SMD:TSOT-23-8_HandSoldering, F.Cu at (104.0, 183.0)
- added U14: TLV9152IDDFR, Package_TO_SOT_SMD:TSOT-23-8_HandSoldering, F.Cu at (73.8, 27.6)
- added U18: TLV9152IDDFR, Package_TO_SOT_SMD:TSOT-23-8_HandSoldering, F.Cu at (157.3, 182.0)
- added U19: TLV743P, Package_TO_SOT_SMD:SOT-23-5_HandSoldering, F.Cu at (81.6, 159.2)
- added U2: USBLC6-2P6, Package_TO_SOT_SMD:SOT-666, F.Cu at (130.7, 62.7)
- added U20: LM4040DBZ-5, Package_TO_SOT_SMD:SOT-23, F.Cu at (37.0, 189.1)
- added U3: IMS330DHCX, Package_LGA:LGA-14_3x2.5mm_P0.5mm_LayoutBorder3x4y, F.Cu at (133.4, 83.5)
- added U4: TLV743P, Package_TO_SOT_SMD:SOT-23-5_HandSoldering, F.Cu at (66.5, 180.4)
- added U5: TLV743P, Package_TO_SOT_SMD:SOT-23-5_HandSoldering, F.Cu at (60.2, 140.1)
- added U6: BD50FC0FP, Package_TO_SOT_SMD:TO-252-2, F.Cu at (175.2, 156.6)
- added U7: LM62440-Q1, Frontbox:IC_LM61460AANRJRR, F.Cu at (181.5, 147.1)
- added U8: MCP2542FDxMF, Package_DFN_QFN:DFN-8-1EP_3x3mm_P0.65mm_EP1.55x2.4mm, F.Cu at (153.1, 100.7)
- added Y1: ABM8G-48.000MHZ, Crystal:Crystal_SMD_Abracon_ABM8G-4Pin_3.2x2.5mm, F.Cu at (118.5, 95.1)
Other:
- board size 60 x 40 mm -> 130 x 100 mm
- board text removed: "Rev: ${REVISION}"

Commit message: Footprints placed, some routing
Parts:
- removed C12, C14: 1uF, Capacitor_SMD:C_0402_1005Metric_Pad0.74x0.62mm_HandSolder
- removed F2: 300mA, Fuse:Fuse_0603_1608Metric_Pad1.05x0.95mm_HandSolder
- removed R75: 220R, Resistor_SMD:R_0402_1005Metric
- removed U4: TLV743P, Package_TO_SOT_SMD:SOT-23-5_HandSoldering
- moved R88 190.0 mm to (188.0, 58.6), turned to -90 degrees
- moved R87 185.1 mm to (186.1, 61.8)
- moved U20 164.0 mm to (162.5, 83.5)
- moved R19 152.1 mm to (161.6, 79.8), turned to -90 degrees
- moved H1 138.9 mm to (16.9, 16.9)
- moved H10 138.9 mm to (22.5, 39.1)
- moved H3 138.9 mm to (16.9, 28.0)
- moved H4 138.9 mm to (16.9, 33.6)
- moved H5 138.9 mm to (16.9, 39.1)
- moved H6 138.9 mm to (22.5, 16.9)
- moved H8 138.9 mm to (22.5, 28.0)
- moved H9 138.9 mm to (22.5, 33.6)
- moved H2 138.9 mm to (16.9, 22.5)
- moved H7 138.9 mm to (22.5, 22.5)
- moved C18 129.9 mm to (176.1, 122.3), turned to 180 degrees
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Connections:
- J3 pad 1: /BRAKE_PRESSURE1 -> /SIG_APPS1
- J3 pad 10: /KILL_KIERA -> /APPS_supply_2_3.3V
- J3 pad 11: GND -> /CAN+
- J3 pad 12: GND -> /CAN-
- J3 pad 13: /CAN+ -> GND
- J3 pad 14: /CAN- -> GND
- J3 pad 15: +5V -> /KILL_PRAWY
- J3 pad 16: +5V -> /BSPD_SENSE
- J3 pad 17: +5V -> /POT_ZAWIAS_1
- J3 pad 18: +24V -> /POT_ZAWIAS2
- J3 pad 19: +24V -> unconnected-(J3-Pin_19-Pad19)
- J3 pad 2: /BRAKE_PRESSURE2 -> /SIG_APPS2
- J3 pad 20: /KILL_PRAWY -> /OVERTRAVEL
- J3 pad 21: /BSPD_SENSE -> +5V
- J3 pad 22: /POT_ZAWIAS2 -> +5V
- J3 pad 23: /POT_ZAWIAS_1 -> +5V
- J3 pad 24: /RTD_BUTTON -> +24V
- J3 pad 25: /APPS_supply_2_3.3V -> +24V
- J3 pad 26: /APPS_supply_1_3.3V -> /SAFE-OUT
- J3 pad 27: /SIG_APPS2 -> /BRAKE_PRESSURE2
- J3 pad 28: /SIG_APPS1 -> /BRAKE_PRESSURE1
- J3 pad 3: GND -> /KILL_LEWY
- J3 pad 4: /SAFE-OUT -> /KILL_KIERA
- J3 pad 8: /OVERTRAVEL -> /RTD_BUTTON
- J3 pad 9: /KILL_LEWY -> /APPS_supply_1_3.3V
- J5 pad 1: /BRAKE_PRESSURE1 -> /SIG_APPS1
- J5 pad 10: /KILL_KIERA -> /APPS_supply_2_3.3V
- J5 pad 11: GND -> /CAN+
- J5 pad 12: GND -> /CAN-
- J5 pad 13: /CAN+ -> GND
- J5 pad 14: /CAN- -> GND
- J5 pad 15: +5V -> /KILL_PRAWY
- J5 pad 16: +5V -> /BSPD_SENSE
- J5 pad 17: +5V -> /POT_ZAWIAS_1
- J5 pad 18: +24V -> /POT_ZAWIAS2
- J5 pad 19: +24V -> unconnected-(J5-Pin_19-Pad19)
- J5 pad 2: /BRAKE_PRESSURE2 -> /SIG_APPS2
- J5 pad 20: /KILL_PRAWY -> /OVERTRAVEL
- J5 pad 21: /BSPD_SENSE -> +5V
- J5 pad 22: /POT_ZAWIAS2 -> +5V
- J5 pad 23: /POT_ZAWIAS_1 -> +5V
- J5 pad 24: /RTD_BUTTON -> +24V
- J5 pad 25: /APPS_supply_2_3.3V -> +24V
- J5 pad 26: /APPS_supply_1_3.3V -> /SAFE-OUT
- J5 pad 27: /SIG_APPS2 -> /BRAKE_PRESSURE2
- J5 pad 28: /SIG_APPS1 -> /BRAKE_PRESSURE1
- J5 pad 3: GND -> /KILL_LEWY
- J5 pad 4: /SAFE-OUT -> /KILL_KIERA
- J5 pad 8: /OVERTRAVEL -> /RTD_BUTTON
- J5 pad 9: /KILL_LEWY -> /APPS_supply_1_3.3V
- U1 pad 36: /DEBUG_LED3 -> /DEBUG_LED4
- U1 pad 37: /DEBUG_LED4 -> /DEBUG_LED3
- U2 pad 1: /USB_EXT_D+ -> /USB_EXT_D-
- U2 pad 3: /USB_EXT_D- -> /USB_EXT_D+
- U2 pad 4: /USB_D- -> /USB_D+
- U2 pad 6: /USB_D+ -> /USB_D-
- U7 pad 1: (no net) -> +7.5V
- U7 pad 10: (no net) -> Net-(U7-SW)
- U7 pad 11: (no net) -> GND
- U7 pad 12: (no net) -> Net-(U7-EN)
- U7 pad 13: (no net) -> Net-(U7-RBOOT)
- U7 pad 14: (no net) -> Net-(U7-CBOOT)
- U7 pad 2: (no net) -> Net-(U7-VCC)
- U7 pad 3: (no net) -> GND
- U7 pad 4: (no net) -> Net-(U7-FB)
- U7 pad 5: (no net) -> unconnected-(U7-PGOOD-Pad5)
- U7 pad 6: (no net) -> GND
- U7 pad 7: (no net) -> Net-(U7-EN)
- U7 pad 8: (no net) -> Net-(U7-EN)
- U7 pad 9: (no net) -> GND
Routing:
- net /EBS_SAFETY: track 0.00 -> 133.1 mm, vias 0 -> 3
- net GND: track 0.00 -> 130.3 mm, vias 0 -> 10
- net /RTD_BUTTON: track 0.00 -> 112.3 mm, vias 0 -> 1
- net /BSPD_SENSE: track 0.00 -> 109.5 mm, vias 0 -> 4
- net /KILL_KIERA: track 0.00 -> 103.1 mm, vias 0 -> 2
- net +5V: track 0.00 -> 96.9 mm
- net /INERTIA: track 0.00 -> 95.5 mm, vias 0 -> 1
- net /OVERTRAVEL: track 0.00 -> 93.3 mm, vias 0 -> 3
- net /CAN-: track 0.00 -> 89.7 mm
- net /CAN+: track 0.00 -> 81.9 mm
- net /SWDIO: track 0.00 -> 72.9 mm, vias 0 -> 1
- net /SAFE-OUT: track 0.00 -> 70.3 mm
- net /NRST: track 0.00 -> 70.2 mm
- net /SAFE-IN: track 0.00 -> 69.7 mm
- net /KILL_PRAWY: track 0.00 -> 66.8 mm, vias 0 -> 2
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- added copper zone on F.Cu, net +5V
- added copper zone on B.Cu, net GND
- added copper zone on F.Cu, net GND
Other:
- outline, holes or cut-outs redrawn
- copper layers 2 -> 4

Commit message: Redid component placement
Parts:
- added C12: 1uF, Capacitor_SMD:C_0402_1005Metric_Pad0.74x0.62mm_HandSolder, F.Cu at (156.3, 104.1)
- added C14: 1uF, Capacitor_SMD:C_0402_1005Metric_Pad0.74x0.62mm_HandSolder, F.Cu at (163.7, 100.5)
- added F2: 300mA, Fuse:Fuse_0603_1608Metric_Pad1.05x0.95mm_HandSolder, F.Cu at (158.1, 104.5)
- added R6: 220R, Resistor_SMD:R_0402_1005Metric_Pad0.72x0.64mm_HandSolder, F.Cu at (242.8, 92.2)
- added R75: 220R, Resistor_SMD:R_0402_1005Metric, F.Cu at (167.5, 107.2)
- added TP3: TestPoint, TestPoint:TestPoint_Pad_1.0x1.0mm, F.Cu at (172.8, 78.5)
- added TP5: TestPoint, TestPoint:TestPoint_Pad_1.0x1.0mm, F.Cu at (142.5, 97.8)
- added U4: TLV743P, Package_TO_SOT_SMD:SOT-23-5_HandSoldering, F.Cu at (163.0, 104.5)
- J2: footprint Connector_PinHeader_1.00mm:PinHeader_1x05_P1.00mm_Vertical -> Connector_PinHeader_2.54mm:PinHeader_1x05_P2.54mm_Vertical
- J4: footprint Connector_USB:USB_C_Receptacle_G-Switch_GT-USB-7010ASV -> Frontbox:CUI_UJ31-CH-31-SMT-TR
- J5: footprint Connector_PinSocket_2.54mm:PinSocket_2x14_P2.54mm_Horizontal -> Connector_PinSocket_2.54mm:PinSocket_2x14_P2.54mm_Vertical
- TP4: value TestPoint_2Pole -> TestPoint; footprint TestPoint:TestPoint_2Pads_Pitch2.54mm_Drill0.8mm -> TestPoint:TestPoint_Pad_1.0x1.0mm
- moved H10 193.4 mm to (197.2, 122.2)
- moved H5 180.8 mm to (197.2, 52.8)
- moved H4 142.4 mm to (128.6, 121.9)
- moved H9 106.7 mm to (127.5, 52.5)
- moved J2 78.4 mm to (147.8, 52.6), turned to -90 degrees
- moved C6 62.4 mm to (109.4, 34.3), turned to -90 degrees
- moved J4 62.3 mm to (135.3, 61.0)
- moved U2 59.8 mm to (138.1, 61.0)
- moved C7 58.4 mm to (112.0, 33.9), turned to 90 degrees
- moved FB1 58.0 mm to (113.6, 33.0)
- moved C10 57.8 mm to (104.8, 44.3)
- moved C23 57.8 mm to (95.9, 48.2)
- moved Y1 57.8 mm to (99.1, 48.1)
- moved C13 57.8 mm to (95.0, 43.2)
- moved C24 57.8 mm to (102.9, 48.2)
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Connections:
- J1 pad 29: GND -> Net-(J1-Pin_29)
- J3 pad 12: /CAN- -> /APPS_supply_1_3.3V
- J3 pad 9: /APPS_supply_1_3.3V -> /CAN-
- J5 pad 12: /CAN- -> /APPS_supply_1_3.3V
- J5 pad 9: /APPS_supply_1_3.3V -> /CAN-
- U2 pad 1: /USB_EXT_D- -> /USB_EXT_D+
- U2 pad 3: /USB_EXT_D+ -> /USB_EXT_D-
- U2 pad 4: /USB_D+ -> /USB_D-
- U2 pad 6: /USB_D- -> /USB_D+
Routing:
- net /BSPD_SENSE: track 109.5 -> 29.6 mm, vias 4 -> 3
- net /OVERTRAVEL: track 93.3 -> 24.5 mm, vias 3 -> 2
- net /SWDIO: track 72.9 -> 6.55 mm, vias 1 -> 0
- net /RTD_BUTTON: track 112.3 -> 50.7 mm, vias 1 -> 0
- net /EBS_SAFETY: track 133.1 -> 73.4 mm, vias 3 -> 1
- net /NRST: track 70.2 -> 16.4 mm
- net /SWCLK: track 58.3 -> 5.03 mm, vias 1 -> 0
- net GND: track 130.3 -> 82.5 mm, vias 10 -> 4
- net /KILL_PRAWY: track 66.8 -> 20.1 mm, vias 2 -> 1
- net /SUSP_R: track 45.0 -> 3.00 mm, vias 2 -> 0
- net /INERTIA: track 95.5 -> 53.9 mm
- net /SAFE-OUT: track 70.3 -> 30.0 mm
- net /KILL_LEWY: track 56.3 -> 16.5 mm, vias 2 -> 1
- net /APPS_sig1: track 41.2 -> 2.32 mm, vias 2 -> 0
- net /Sense_left: track 42.5 -> 4.16 mm
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- removed copper zone on F.Cu, net GND
Other:
- board size 130 x 100 mm -> 140 x 75 mm
- board text added: "3v3"
- board text added: "5v ref"
- board text added: "APPS res"
- board text added: "Apps res"
- board text added: "CLK"
- board text added: "DIO"
- board text added: "GND"
- board text added: "H"
- board text added: "L"
- board text added: "NRST"
- board text added: "RX"
- board text added: "SCL"
- board text added: "SDA"
- board text added: "Speed"
- board text added: "TX"
- board text added: "Yaw"

Commit message: Finished most of the routing
Parts:
- added G***: LOGO, Logos:PUTM_LOGO_15mm, F.Cu at (151.8, 137.9)
- added G***: LOGO, Logos:SignatureBox25mm, B.Cu at (162.2, 119.0)
- moved R5 74.5 mm to (150.7, 73.6)
- moved R1 74.2 mm to (152.0, 73.6)
- moved R2 74.2 mm to (153.3, 73.6)
- moved D5 74.1 mm to (150.4, 69.9), turned to 180 degrees
- moved R3 74.1 mm to (154.6, 73.6)
- moved R4 74.0 mm to (155.9, 73.6)
- moved D1 72.3 mm to (150.4, 68.8), turned to 180 degrees
- moved D2 70.8 mm to (150.5, 67.4), turned to 180 degrees
- moved C6 70.2 mm to (160.2, 82.7)
- moved C7 69.5 mm to (161.6, 82.7), turned to -90 degrees
- moved C10 69.4 mm to (155.9, 91.2)
- moved C23 69.4 mm to (147.0, 95.1)
- moved C24 69.4 mm to (154.0, 95.1)
- moved U1 69.4 mm to (152.2, 83.5)
- moved C13 69.4 mm to (146.2, 90.1)
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Connections:
- J3 pad 27: /BRAKE_PRESSURE2 -> /BRAKE_PRESSURE1
- J3 pad 28: /BRAKE_PRESSURE1 -> /BRAKE_PRESSURE2
- J5 pad 27: /BRAKE_PRESSURE2 -> unconnected-(J5-Pin_27-Pad27)
- U1 pad 10: /Sense_right -> /Sense_driver
- U1 pad 11: /Sense_left -> /Sense_inertia
- U1 pad 12: /Sense_EBS -> /Safety_control
- U1 pad 17: /APPS_sig1 -> /APPS_sig2
- U1 pad 18: /APPS_sig2 -> /APPS_sig1
- U1 pad 2: /Safety_control -> /Sense_overtravel
- U1 pad 20: /SUSP_R -> /SUSP_L
- U1 pad 21: /SUSP_L -> /SUSP_R
- U1 pad 22: /Brake_pressure_rear -> /Brake_pressure_front
- U1 pad 23: /Brake_pressure_front -> /Brake_pressure_rear
- U1 pad 3: /Sense_BSPD -> /RTD_BUTTON_sig
- U1 pad 4: /Sense_overtravel -> /Sense_EBS
- U1 pad 62: /RTD_BUTTON_sig -> /Sense_BSPD
- U1 pad 8: /Sense_inertia -> /Sense_left
- U1 pad 9: /Sense_driver -> /Sense_right
Routing:
- net /OVERTRAVEL: track 24.5 -> 107.1 mm, vias 2 -> 3
- net /BSPD_SENSE: track 29.6 -> 107.4 mm
- net +5V: track 81.7 -> 152.7 mm, vias 0 -> 2
- net /NRST: track 16.4 -> 77.2 mm
- net 5v_ref: track 5.62 -> 63.3 mm, vias 1 -> 4
- net /Safety_control: track 5.66 -> 61.3 mm, vias 0 -> 2
- net /CAN-: track 63.0 -> 114.0 mm, vias 0 -> 2
- net /RTD_BUTTON: track 50.7 -> 99.8 mm, vias 0 -> 2
- net /CAN+: track 56.5 -> 105.6 mm, vias 0 -> 2
- net /YAWPROBE_I^{2}C_SDA: track 0.73 -> 45.9 mm
- net /EBS_SAFETY: track 73.4 -> 118.4 mm, vias 1 -> 2
- net /SAFE-OUT: track 30.0 -> 73.0 mm
- net /YAWPROBE_I^{2}C_SCL: track 0.75 -> 40.9 mm
- net /Sense_BSPD: track 3.68 -> 43.5 mm
- net /SWDIO: track 6.55 -> 45.9 mm, vias 0 -> 1
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Other:
- outline, holes or cut-outs redrawn
- board text added: "Szymon Kostrubiec"
- board text added: "We do these things not because they're easy, but because we thought they were going to be."

Commit message: Layout mostly done
Parts:
- moved H7 260.0 mm to (262.5, 122.5)
- moved H8 241.3 mm to (262.5, 52.5)
- moved H2 237.6 mm to (232.5, 122.5)
- moved H3 216.9 mm to (232.5, 52.5)
- moved G*** 31.8 mm to (152.2, 106.1)
- moved C3 7.13 mm to (165.3, 88.9), turned to 0 degrees
- moved FB6 1.35 mm to (164.4, 93.2), turned to 0 degrees
- moved C35 1.17 mm to (178.2, 107.2)
- moved C4 0.44 mm to (165.3, 90.6), turned to 90 degrees
Routing:
- net +5V: track 152.7 -> 271.0 mm, vias 2 -> 6
- net GND: track 80.5 -> 29.6 mm, vias 3 -> 6
- net /EBS_SAFETY: track 118.4 -> 77.0 mm
- net +3.3V: track 61.5 -> 102.3 mm, vias 0 -> 17
- net /KILL_KIERA: track 94.2 -> 61.7 mm, vias 2 -> 1
- net /SIG_APPS1: track 71.4 -> 39.4 mm
- net /NRST: track 77.2 -> 100.9 mm, vias 0 -> 2
- net /APPS_supply_2_3.3V: track 53.0 -> 35.3 mm
- net /POT_ZAWIAS2: track 57.0 -> 41.1 mm, vias 1 -> 0
- net /KILL_LEWY: track 43.5 -> 55.2 mm
- net Net-(IC2-VS): track 0.00 -> 10.7 mm, vias 0 -> 1
- net Net-(IC1-VS): track 0.00 -> 9.12 mm
- net /SAFE-IN: track 67.3 -> 60.3 mm, vias 0 -> 1
- net /OVERTRAVEL: track 107.1 -> 101.4 mm, vias 3 -> 1
- net Net-(U3-VDD): track 1.73 -> 5.69 mm
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- added copper zone on In2.Cu, net +3.3V
- added copper zone on F.Cu, net GND
- added copper zone on In1.Cu, net GND
- added copper zone on In2.Cu, net GND
Other:
- outline, holes or cut-outs redrawn
- board text added: "locked"
- board text removed: "Apps res"

Commit message: Ready for production
Parts:
- moved G*** 15.4 mm to (157.2, 104.5)
- moved C15 11.9 mm to (162.1, 55.3)
- moved R6 2.32 mm to (241.6, 94.2), turned to 0 degrees
- moved G*** 1.96 mm to (150.5, 105.1)
- moved C8 1.71 mm to (159.8, 79.1)
- moved J1 1.51 mm to (252.4, 88.0)
- moved J3 1.51 mm to (234.8, 105.4)
- moved FB1 1.23 mm to (161.5, 79.4)
- moved J4 0.79 mm to (135.4, 61.7)
- moved U2 0.79 mm to (138.2, 61.7)
- moved C3 0.20 mm to (165.3, 88.7)
- moved R73 0.15 mm to (172.0, 104.1)
Connections:
- J3 pad 27: /BRAKE_PRESSURE1 -> /BRAKE_PRESSURE2
- J3 pad 28: /BRAKE_PRESSURE2 -> /BRAKE_PRESSURE1
- J5 pad 27: unconnected-(J5-Pin_27-Pad27) -> /BRAKE_PRESSURE2
Routing:
- net /APPS_supply_2_3.3V: track 35.3 -> 52.2 mm
- net /Safety_control: track 61.3 -> 50.7 mm, vias 2 -> 0
- net /SWCLK: track 42.5 -> 49.2 mm
- net Net-(U7-EN): track 46.2 -> 51.7 mm
- net GND: track 29.6 -> 34.2 mm, vias 6 -> 9
- net +7.5V: track 49.8 -> 54.1 mm
- net +5V: track 271.0 -> 266.9 mm
- net Net-(U8-VDD): track 2.93 -> 7.00 mm
- net /CAN+: track 104.8 -> 108.5 mm
- net Net-(U6-VCC): track 15.7 -> 12.6 mm
- net /CAN-: track 110.3 -> 113.2 mm
- net /BSPD_SENSE: track 105.8 -> 103.4 mm
- net /OVERTRAVEL: track 101.4 -> 99.1 mm
- net Net-(U3-VDD): track 5.69 -> 7.67 mm
- net /SUSP_R: track 34.8 -> 32.9 mm
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Other:
- board text added: "Apps res"
- board text added: "{dblquote}We do these things not because they're easy, but because we thought they were going to be.{dblquote}"
- board text removed: "We do these things not because they're easy, but because we thought they were going to be."
- board text removed: "locked"
