File: Hardware/PUTM_EV_Frontbox_2023/PUTM_EV_Frontbox_2023.kicad_pcb (KiCad board)
At the start: 4 copper layers, 140 x 75 mm, 171 parts, among them IC1 ELVH-MF12D-HRRJ-C-N3A4, IC2 ELVH-MF12D-HRRJ-C-N3A4, J1 Złącze TE, J2 Conn_01x04, J3 Conn_02x14_Counter_Clockwise, J4 USB_C_Receptacle, J5 Conn_02x14_Counter_Clockwise, K1 UMS05-1A80-75D, Q1 NX7002AK, SW1 Reset switch, U1 STM32G473RCTx, U10 TLP291-4, U11 TLP291-4, U12 TLV9152IDDFR, U13 TLV9152IDDFR, U14 TLV9152IDDFR, U18 TLV9152IDDFR, U19 TLV743P, U2 USBLC6-2P6, U20 LM4040DBZ-5, U3 IMS330DHCX, U4 TLV743P, U5 TLV743P, U6 BD50FC0FP, U7 LM62440-Q1, U8 MCP2542FDxMF, Y1 ABM8G-48.000MHZ

Commit message: PCB taken apart
Parts:
- removed C1: 100nF, Capacitor_SMD:C_0402_1005Metric_Pad0.74x0.62mm_HandSolder
- removed C26, C27, C33, C34: 47n 1%, Capacitor_SMD:C_0402_1005Metric_Pad0.74x0.62mm_HandSolder
- removed C28, C29, C35: 100n, Capacitor_SMD:C_0402_1005Metric_Pad0.74x0.62mm_HandSolder
- removed C39: 10uF, Capacitor_SMD:CP_Elec_4x5.7
- removed G***: LOGO, Logos:PUTM_LOGO_15mm
- removed G***: LOGO, Logos:SignatureBox25mm
- removed J1: Złącze TE, Frontbox:Autosport
- removed J3: Conn_02x14_Counter_Clockwise, Connector_PinHeader_2.54mm:PinHeader_2x14_P2.54mm_Horizontal
- removed J4: USB_C_Receptacle, Frontbox:CUI_UJ31-CH-31-SMT-TR
- removed R30, R31, R34, R35, R36, R37, R38, R39, R40, R41, R42, R43, R44, R45, R46, R47: R_Small, Resistor_SMD:R_0402_1005Metric
- removed R32, R33: 10k 1%, Resistor_SMD:R_0402_1005Metric
- removed R48: 10k, Resistor_SMD:R_0402_1005Metric
- removed R6: 220R, Resistor_SMD:R_0402_1005Metric_Pad0.72x0.64mm_HandSolder
- removed SW1: Reset switch, Button_Switch_SMD:SW_MEC_5GSH9
- removed U13, U14: TLV9152IDDFR, Package_TO_SOT_SMD:TSOT-23-8_HandSoldering
- added C48: 100n, Capacitor_SMD:C_0603_1608Metric_Pad1.08x0.95mm_HandSolder, F.Cu at (217.8, 68.6)
- added C49: 100n, Capacitor_SMD:C_0603_1608Metric_Pad1.08x0.95mm_HandSolder, F.Cu at (238.2, 46.6)
- added C50: 100n, Capacitor_SMD:C_0603_1608Metric_Pad1.08x0.95mm_HandSolder, F.Cu at (238.2, 49.2)
- added C51: 10n, Capacitor_SMD:C_0603_1608Metric_Pad1.08x0.95mm_HandSolder, F.Cu at (238.2, 51.7)
- added C52: 10n, Capacitor_SMD:C_0603_1608Metric_Pad1.08x0.95mm_HandSolder, F.Cu at (238.2, 54.2)
- added C53: 100n, Capacitor_SMD:C_0603_1608Metric_Pad1.08x0.95mm_HandSolder, F.Cu at (238.2, 56.7)
- added C54: 100n, Capacitor_SMD:C_0603_1608Metric_Pad1.08x0.95mm_HandSolder, F.Cu at (242.5, 46.6)
- added C55: 100n, Capacitor_SMD:C_0603_1608Metric_Pad1.08x0.95mm_HandSolder, F.Cu at (217.8, 46.6)
- added C56: 100n, Capacitor_SMD:C_0603_1608Metric_Pad1.08x0.95mm_HandSolder, F.Cu at (217.8, 49.2)
- added C57: 10n, Capacitor_SMD:C_0603_1608Metric_Pad1.08x0.95mm_HandSolder, F.Cu at (217.8, 51.7)
- added C58: 10n, Capacitor_SMD:C_0603_1608Metric_Pad1.08x0.95mm_HandSolder, F.Cu at (217.8, 54.2)
- added C59: 100n, Capacitor_SMD:C_0603_1608Metric_Pad1.08x0.95mm_HandSolder, F.Cu at (217.8, 56.7)
- added C60: 100n, Capacitor_SMD:C_0603_1608Metric_Pad1.08x0.95mm_HandSolder, F.Cu at (222.2, 46.6)
- added D10: 24V, Diode_SMD:D_0603_1608Metric_Pad1.05x0.95mm_HandSolder, F.Cu at (231.1, 63.7)
- added D9: 24V, Diode_SMD:D_0603_1608Metric_Pad1.05x0.95mm_HandSolder, F.Cu at (251.4, 63.7)
- added JP3: POT/DAC, Jumper:SolderJumper-3_P1.3mm_Bridged12_RoundedPad1.0x1.5mm, F.Cu at (246.4, 59.7)
- added JP4: POT/DAC, Jumper:SolderJumper-3_P1.3mm_Bridged12_RoundedPad1.0x1.5mm, F.Cu at (226.0, 59.7)
- added R57: 220R, Resistor_SMD:R_0402_1005Metric, F.Cu at (156.9, 41.3)
- added R61: 100R, Resistor_SMD:R_0603_1608Metric_Pad0.98x0.95mm_HandSolder, F.Cu at (217.8, 71.1)
- added R62: 0R, Resistor_SMD:R_0603_1608Metric_Pad0.98x0.95mm_HandSolder, F.Cu at (217.8, 73.6)
- added R63: 100R, Resistor_SMD:R_0603_1608Metric_Pad0.98x0.95mm_HandSolder, F.Cu at (217.8, 76.1)
- added R64: 0R, Resistor_SMD:R_0603_1608Metric_Pad0.98x0.95mm_HandSolder, F.Cu at (217.8, 78.6)
- added R65: 3k3, Resistor_SMD:R_0603_1608Metric_Pad0.98x0.95mm_HandSolder, F.Cu at (217.8, 81.1)
- added R66: 0R, Resistor_SMD:R_0603_1608Metric_Pad0.98x0.95mm_HandSolder, F.Cu at (217.8, 83.6)
- added R78: 33k, Resistor_SMD:R_0603_1608Metric_Pad0.98x0.95mm_HandSolder, F.Cu at (222.2, 49.2)
- added R90: 100k, Resistor_SMD:R_0603_1608Metric_Pad0.98x0.95mm_HandSolder, F.Cu at (222.2, 51.7)
- added R91: 0R, Resistor_SMD:R_0603_1608Metric_Pad0.98x0.95mm_HandSolder, F.Cu at (222.2, 54.2)
- added R92: 4k7, Resistor_SMD:R_0603_1608Metric_Pad0.98x0.95mm_HandSolder, F.Cu at (222.2, 56.7)
- added R94: 4k7, Resistor_SMD:R_0603_1608Metric_Pad0.98x0.95mm_HandSolder, F.Cu at (226.5, 49.2)
- added R95: 4k7, Resistor_SMD:R_0603_1608Metric_Pad0.98x0.95mm_HandSolder, F.Cu at (226.5, 51.7)
- added RV3: 2k, Potentiometer_SMD:Potentiometer_Bourns_3214J_Horizontal, F.Cu at (237.1, 70.5)
- added RV5: 2k, Potentiometer_SMD:Potentiometer_Bourns_3214J_Horizontal, F.Cu at (223.8, 70.5)
- added RV6: 1k, Potentiometer_SMD:Potentiometer_Bourns_3214J_Horizontal, F.Cu at (239.8, 61.1)
- added RV7: 1k, Potentiometer_SMD:Potentiometer_Bourns_3214J_Horizontal, F.Cu at (219.4, 61.1)
- added TP14: BR_N, TestPoint:TestPoint_Pad_D1.0mm, F.Cu at (231.8, 68.8)
- added TP15: BR_P, TestPoint:TestPoint_Pad_D1.0mm, F.Cu at (231.8, 71.9)
- added TP16: BR_MID, TestPoint:TestPoint_Pad_D1.0mm, F.Cu at (231.8, 75.0)
- added TP17: BR_OUT, TestPoint:TestPoint_Pad_D1.0mm, F.Cu at (231.8, 78.0)
- added TP22: BR_N, TestPoint:TestPoint_Pad_D1.0mm, F.Cu at (221.5, 75.2)
- added TP23: BR_P, TestPoint:TestPoint_Pad_D1.0mm, F.Cu at (221.5, 78.2)
- added TP24: BR_MID, TestPoint:TestPoint_Pad_D1.0mm, F.Cu at (221.5, 81.3)
- added TP25: BR_OUT, TestPoint:TestPoint_Pad_D1.0mm, F.Cu at (221.5, 84.3)
- added TP26: APPS_P, TestPoint:TestPoint_Pad_D1.0mm, F.Cu at (250.6, 46.9)
- added TP27: APPS_N, TestPoint:TestPoint_Pad_D1.0mm, F.Cu at (250.6, 50.0)
- added TP28: APPS_MID, TestPoint:TestPoint_Pad_D1.0mm, F.Cu at (250.6, 53.0)
- added TP29: APPS_OUT, TestPoint:TestPoint_Pad_D1.0mm, F.Cu at (250.6, 56.1)
- added TP30: APPS_P, TestPoint:TestPoint_Pad_D1.0mm, F.Cu at (230.2, 46.9)
- added TP31: APPS_N, TestPoint:TestPoint_Pad_D1.0mm, F.Cu at (230.2, 50.0)
- added TP32: APPS_MID, TestPoint:TestPoint_Pad_D1.0mm, F.Cu at (230.2, 53.0)
- added TP33: APPS_OUT, TestPoint:TestPoint_Pad_D1.0mm, F.Cu at (230.2, 56.1)
- added U17: MCP6002-xMC, Package_DFN_QFN:DFN-8-1EP_3x2mm_P0.5mm_EP1.7x1.4mm, F.Cu at (225.7, 75.5)
- added U21: MCP6001, Package_TO_SOT_SMD:SOT-23-5, F.Cu at (251.8, 60.2)
- added U22: MCP6N11-005, Package_DFN_QFN:TDFN-8-1EP_3x2mm_P0.5mm_EP1.3x1.4mm, F.Cu at (225.8, 63.5)
- added U23: MCP6001, Package_TO_SOT_SMD:SOT-23-5, F.Cu at (231.4, 60.2)
- R67: value R_Small -> 10k; footprint Resistor_SMD:R_0402_1005Metric -> Resistor_SMD:R_0603_1608Metric_Pad0.98x0.95mm_HandSolder
- R68: value R_Small -> 33k; footprint Resistor_SMD:R_0402_1005Metric -> Resistor_SMD:R_0603_1608Metric_Pad0.98x0.95mm_HandSolder
- R69: value 10k 1% -> 100k; footprint Resistor_SMD:R_0402_1005Metric -> Resistor_SMD:R_0603_1608Metric_Pad0.98x0.95mm_HandSolder
- R70: value 10k 1% -> 0R; footprint Resistor_SMD:R_0402_1005Metric -> Resistor_SMD:R_0603_1608Metric_Pad0.98x0.95mm_HandSolder
- R71, R73, R74: value R_Small -> 4k7; footprint Resistor_SMD:R_0402_1005Metric -> Resistor_SMD:R_0603_1608Metric_Pad0.98x0.95mm_HandSolder
- R72: value R_Small -> 1k; footprint Resistor_SMD:R_0402_1005Metric -> Resistor_SMD:R_0603_1608Metric_Pad0.98x0.95mm_HandSolder
- R75: value 220R -> 10k; footprint Resistor_SMD:R_0402_1005Metric -> Resistor_SMD:R_0603_1608Metric_Pad0.98x0.95mm_HandSolder
- R93: value 2k -> 1k; footprint Resistor_SMD:R_0402_1005Metric -> Resistor_SMD:R_0603_1608Metric_Pad0.98x0.95mm_HandSolder
- U18: value TLV9152IDDFR -> MCP6N11-005; footprint Package_TO_SOT_SMD:TSOT-23-8_HandSoldering -> Package_DFN_QFN:TDFN-8-1EP_3x2mm_P0.5mm_EP1.3x1.4mm
- U2: value USBLC6-2P6 -> MCP6002-xMC; footprint Package_TO_SOT_SMD:SOT-666 -> Package_DFN_QFN:DFN-8-1EP_3x2mm_P0.5mm_EP1.7x1.4mm
- moved H7 139.4 mm to (158.2, 30.0)
- moved H2 127.5 mm to (158.2, 18.9)
- moved C25 111.0 mm to (98.2, 150.0)
- moved R22 111.0 mm to (100.8, 156.2)
- moved R23 111.0 mm to (104.4, 150.5)
- moved R29 111.0 mm to (99.2, 146.3)
- moved R76 111.0 mm to (104.6, 155.0)
- moved R17 111.0 mm to (96.6, 158.3)
- moved R18 111.0 mm to (101.8, 145.5)
- moved R21 111.0 mm to (101.3, 158.2)
- moved R24 111.0 mm to (103.0, 155.2)
- moved R25 111.0 mm to (103.2, 149.8)
- moved R26 111.0 mm to (98.4, 158.3)
- moved R27 111.0 mm to (101.3, 147.2)
- moved R28 111.0 mm to (97.9, 154.8)
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Connections:
- C14 pad 1: Net-(U4-OUT) -> /APPS1_3V3
- C38 pad 1: /APPS_supply_2_3.3V -> /APPS2_3V3
- J2 pad 1: +3.3V -> unconnected-(J2-Pin_1-Pad1)
- J2 pad 2: /SWCLK -> unconnected-(J2-Pin_2-Pad2)
- J2 pad 3: GND -> unconnected-(J2-Pin_3-Pad3)
- J2 pad 4: /SWDIO -> unconnected-(J2-Pin_4-Pad4)
- J2 pad 5: /NRST -> +3.3V
- J5 pad 1: /SIG_APPS1 -> /BSPD_SENSE
- J5 pad 10: /APPS_supply_2_3.3V -> Net-(J5-Pin_10)
- J5 pad 11: /CAN+ -> Net-(J5-Pin_11)
- J5 pad 12: /APPS_supply_1_3.3V -> /BRAKE_PRESSURE1
- J5 pad 13: GND -> /BRAKE_PRESSURE2
- J5 pad 14: GND -> /POT_ZAWIAS2
- J5 pad 15: /KILL_PRAWY -> /POT_ZAWIAS_1
- J5 pad 16: /BSPD_SENSE -> /APPS_POT_2
- J5 pad 17: /POT_ZAWIAS_1 -> /APPS_POT_1
- J5 pad 18: /POT_ZAWIAS2 -> Net-(J5-Pin_18)
- J5 pad 19: unconnected-(J5-Pin_19-Pad19) -> Net-(J5-Pin_19)
- J5 pad 2: /SIG_APPS2 -> /KILL_PRAWY
- J5 pad 20: /OVERTRAVEL -> unconnected-(J5-Pin_20-Pad20)
- J5 pad 21: +5V -> unconnected-(J5-Pin_21-Pad21)
- J5 pad 22: +5V -> unconnected-(J5-Pin_22-Pad22)
- J5 pad 23: +5V -> /CAN+
- J5 pad 24: +24V -> /CAN-
- J5 pad 25: +24V -> GND
- J5 pad 26: /SAFE-OUT -> GND
- J5 pad 27: /BRAKE_PRESSURE2 -> +5V
- J5 pad 28: /BRAKE_PRESSURE1 -> +24V
- J5 pad 3: /KILL_LEWY -> /OVERTRAVEL
- J5 pad 4: /KILL_KIERA -> /KILL_LEWY
- J5 pad 5: /SAFE-IN -> /KILL_KIERA
- J5 pad 8: /RTD_BUTTON -> /SAFE-IN
- J5 pad 9: /CAN- -> /SAFE-OUT
- R67 pad 1: 5v_ref -> 3V3_POT1
- R67 pad 2: /APPS measurement1/OFFSET -> Net-(R67-Pad2)
- R68 pad 1: /APPS measurement1/OFFSET -> Net-(R68-Pad1)
- R69 pad 1: /SIG_APPS2 -> /APPS1/POT2
- R69 pad 2: Net-(C34-Pad1) -> GND
- R70 pad 1: Net-(C34-Pad1) -> Net-(U18-EN)
- R70 pad 2: Net-(U18A-+) -> 3V3_POT1
- R71 pad 1: Net-(U18B-+) -> Net-(U18-FG)
- R71 pad 2: Net-(U18A--) -> Net-(R71-Pad2)
- R72 pad 1: Net-(U18B-+) -> GND
- R72 pad 2: GND -> Net-(U18-FG)
- R73 pad 1: Net-(U18B--) -> Net-(R71-Pad2)
- R73 pad 2: /APPS measurement1/OFFSET -> Net-(C54-Pad1)
- R74 pad 1: /APPS_sig2 -> Net-(C54-Pad1)
- R74 pad 2: Net-(U18B--) -> Net-(U21-+)
- R75 pad 1: Net-(U4-OUT) -> 3V3_POT1
- R75 pad 2: /APPS_supply_1_3.3V -> Net-(R75-Pad2)
- R93 pad 1: /RTD_BUTTON -> GND
- R93 pad 2: Net-(R93-Pad2) -> Net-(U22-FG)
- U1 pad 44: unconnected-(U1-PA10-Pad44) -> /DAC1_REF
- U1 pad 45: /USB_D- -> unconnected-(U1-PA11-Pad45)
- U1 pad 46: /USB_D+ -> unconnected-(U1-PA12-Pad46)
- U1 pad 52: unconnected-(U1-PC10-Pad52) -> /DAC2_REF
- U11 pad 11: GND -> (no net)
- U11 pad 12: /RTD_BUTTON_sig -> (no net)
- U11 pad 5: Net-(R93-Pad2) -> (no net)
- U11 pad 6: GND -> (no net)
- U18 pad 1: Net-(U18A--) -> Net-(U18-FG)
- U18 pad 2: Net-(U18A--) -> Net-(JP3-C)
- U18 pad 3: Net-(U18A-+) -> /APPS1/POT2
- U18 pad 5: Net-(U18B-+) -> GND
- U18 pad 6: Net-(U18B--) -> Net-(R71-Pad2)
- U18 pad 7: /APPS_sig2 -> 3V3_POT1
- U18 pad 8: +3.3V -> Net-(U18-EN)
- U2 pad 1: /USB_EXT_D+ -> /Brake_press_front
- U2 pad 2: GND -> Net-(U2A--)
- U2 pad 3: /USB_EXT_D- -> Net-(U2A-+)
- U2 pad 4: /USB_D- -> GND
- U2 pad 5: +5V -> Net-(U2B-+)
- U2 pad 6: /USB_D+ -> Net-(U2B--)
- U4 pad 5: Net-(U4-OUT) -> /APPS1_3V3
- U5 pad 5: /APPS_supply_2_3.3V -> /APPS2_3V3
Routing:
- net /RTD_BUTTON: track 100.9 -> 0.00 mm, vias 1 -> 0
- net (no net): track 0.00 -> 95.9 mm
- net +5V: track 266.9 -> 177.6 mm, vias 6 -> 3
- net /NRST: track 100.8 -> 23.1 mm, vias 2 -> 1
- net /BSPD_SENSE: track 103.4 -> 47.3 mm
- net /APPS_supply_2_3.3V: track 52.2 -> 0.00 mm
- net /SAFE-IN: track 60.5 -> 111.4 mm
- net +3.3V: track 102.5 -> 53.4 mm, vias 17 -> 11
- net /APPS_supply_1_3.3V: track 48.1 -> 0.00 mm, vias 1 -> 0
- net /OVERTRAVEL: track 99.1 -> 51.7 mm, vias 1 -> 0
- net unconnected-(J5-Pin_20-Pad20): track 0.00 -> 45.5 mm, vias 0 -> 1
- net /INERTIA: track 81.0 -> 38.0 mm, vias 2 -> 1
- net unconnected-(J2-Pin_4-Pad4): track 0.00 -> 42.1 mm
- net /SWDIO: track 45.9 -> 3.86 mm
- net +3V3: track 0.00 -> 40.9 mm
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- removed copper zone on In2.Cu, net GND
Other:
- board size 140 x 75 mm -> 75 x 75 mm
- board text removed: "5v ref"
- board text removed: "APPS res"
- board text removed: "Apps res"
- board text removed: "H"
- board text removed: "L"
- board text removed: "RX"
- board text removed: "Speed"
- board text removed: "TX"
- board text removed: "Yaw"

Commit message: Updated PCB
Parts:
- added C1: 100nF, Capacitor_SMD:C_0402_1005Metric_Pad0.74x0.62mm_HandSolder, F.Cu at (47.7, 68.6)
- added C29: 100n, Capacitor_SMD:C_0603_1608Metric_Pad1.08x0.95mm_HandSolder, F.Cu at (30.3, 55.9)
- added R38: 100R, Resistor_SMD:R_0603_1608Metric_Pad0.98x0.95mm_HandSolder, F.Cu at (30.3, 58.4)
- added R39: 0R, Resistor_SMD:R_0603_1608Metric_Pad0.98x0.95mm_HandSolder, F.Cu at (30.3, 60.9)
- added R40: 100R, Resistor_SMD:R_0603_1608Metric_Pad0.98x0.95mm_HandSolder, F.Cu at (30.3, 63.4)
- added R41: 0R, Resistor_SMD:R_0603_1608Metric_Pad0.98x0.95mm_HandSolder, F.Cu at (30.3, 65.9)
- added R42: 3k3, Resistor_SMD:R_0603_1608Metric_Pad0.98x0.95mm_HandSolder, F.Cu at (30.3, 68.5)
- added R43: 0R, Resistor_SMD:R_0603_1608Metric_Pad0.98x0.95mm_HandSolder, F.Cu at (30.3, 71.0)
- added R48: 220R, Resistor_SMD:R_0402_1005Metric, F.Cu at (51.9, 57.6)
- added R57: 220R, Resistor_SMD:R_0402_1005Metric, F.Cu at (51.9, 59.6)
- added R58: 220R, Resistor_SMD:R_0402_1005Metric, F.Cu at (51.9, 61.6)
- added R6: 220R, Resistor_SMD:R_0402_1005Metric, F.Cu at (51.9, 55.6)
- added SW1: Reset switch, Button_Switch_SMD:SW_MEC_5GSH9, F.Cu at (40.3, 63.0)
- D1, D2, D3, D4, D5: footprint LED_SMD:LED_0201_0603Metric -> Diode_SMD:D_0603_1608Metric_Pad1.05x0.95mm_HandSolder
- R1, R2, R3, R4, R5: footprint Resistor_SMD:R_0402_1005Metric -> Resistor_SMD:R_0603_1608Metric_Pad0.98x0.95mm_HandSolder
- moved H1 129.9 mm to (146.8, 17.8)
- moved H6 129.9 mm to (152.4, 17.8)
- moved D1 49.4 mm to (59.0, 77.7), turned to 90 degrees
- moved D2 48.6 mm to (60.7, 77.7), turned to 90 degrees
- moved D3 47.9 mm to (62.3, 77.7), turned to 90 degrees
- moved D4 47.4 mm to (63.9, 77.7), turned to 90 degrees
- moved D5 43.1 mm to (65.6, 77.7), turned to 90 degrees
- moved R85 8.75 mm to (44.8, 96.3)
- moved R86 8.75 mm to (46.2, 96.3)
- moved R1 8.73 mm to (59.0, 81.1), turned to 90 degrees
- moved R2 8.57 mm to (60.7, 81.1), turned to 90 degrees
- moved R3 8.39 mm to (62.3, 81.1), turned to 90 degrees
- moved R4 8.21 mm to (64.0, 81.1), turned to 90 degrees
- moved R5 7.93 mm to (65.5, 81.1), turned to 90 degrees
- moved FB4 3.09 mm to (51.1, 91.2), turned to 90 degrees
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Connections:
- J2 pad 1: unconnected-(J2-Pin_1-Pad1) -> +3.3V
- J2 pad 2: unconnected-(J2-Pin_2-Pad2) -> /SWCLK
- J2 pad 3: unconnected-(J2-Pin_3-Pad3) -> GND
- J2 pad 4: unconnected-(J2-Pin_4-Pad4) -> /SWDIO
- J2 pad 5: +3.3V -> /NRST
Routing:
- net +5V: track 177.6 -> 0.00 mm, vias 3 -> 0
- net /SAFE-IN: track 111.4 -> 0.00 mm, vias 1 -> 0
- net (no net): track 95.9 -> 0.00 mm
- net /CAN-: track 85.2 -> 0.00 mm
- net /CAN+: track 82.4 -> 0.00 mm
- net /EBS_SAFETY: track 76.4 -> 0.00 mm, vias 1 -> 0
- net /SAFE-OUT: track 73.2 -> 0.00 mm
- net /BRAKE_PRESSURE1: track 60.0 -> 0.00 mm
- net +24V: track 58.3 -> 0.00 mm
- net +7.5V: track 52.5 -> 0.00 mm, vias 1 -> 0
- net Net-(U7-EN): track 51.7 -> 0.00 mm
- net /OVERTRAVEL: track 51.7 -> 0.00 mm
- net +3.3V: track 53.4 -> 1.80 mm, vias 11 -> 0
- net /KILL_LEWY: track 48.5 -> 0.00 mm, vias 1 -> 0
- net /BSPD_SENSE: track 47.3 -> 0.00 mm
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- removed copper zone on In2.Cu, net +3.3V
- removed copper zone on F.Cu, net +5V
- removed copper zone on B.Cu, net GND
- removed copper zone on F.Cu, net GND
- removed copper zone on In1.Cu, net GND
Other:
- board text removed: "Szymon Kostrubiec"
- board text removed: "{dblquote}We do these things not because they're easy, but because we thought they were going to be.{dblquote}"
