File: Hardware/imu_sensor.kicad_sch (KiCad schematic)
At the start: 6 parts

Commit message: Frontbox 2025 Version 1.0
Connections:
- no-connect marks 2 -> 3
Changed lines of the file:
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@@
+	)
+	(no_connect
+		(at 93.98 85.09)
 	)
 	(no_connect
