File: Hardware/suspension_potentiometer.kicad_sch (KiCad schematic)
At the start: 18 parts, among them U16 MCP6N11-005, U17 MCP6001

Commit message: Changes in current layout, added tensometers to layout
Parts:
- U16: footprint Package_DFN_QFN:TDFN-8-1EP_3x2mm_P0.5mm_EP1.80x1.65mm -> Samacsys:TDFN-8-1EP_3x2mm_P0.5mm_EP1.70x1.65mm
Changed lines of the file:
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@@
 			)
 		)
-		(property "Footprint" "Package_DFN_QFN:TDFN-8-1EP_3x2mm_P0.5mm_EP1.80x1.65mm"
+		(property "Footprint" "Samacsys:TDFN-8-1EP_3x2mm_P0.5mm_EP1.70x1.65mm"
 			(at 113.03 109.855 0)
 			(effects

Commit message: Changes in power section
Parts:
- TP13, TP14, TP15, TP16: footprint TestPoint:TestPoint_Pad_D1.0mm -> TestPoint:TestPoint_THTPad_D1.0mm_Drill0.5mm
Changed lines of the file:
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@@
 			)
 		)
-		(property "Footprint" "TestPoint:TestPoint_Pad_D1.0mm"
+		(property "Footprint" "TestPoint:TestPoint_THTPad_D1.0mm_Drill0.5mm"
 			(at 133.35 86.995 0)
 			(effects
@@
 			)
 		)
-		(property "Footprint" "TestPoint:TestPoint_Pad_D1.0mm"
+		(property "Footprint" "TestPoint:TestPoint_THTPad_D1.0mm_Drill0.5mm"
 			(at 133.35 92.075 0)
 			(effects
@@
 			)
 		)
-		(property "Footprint" "TestPoint:TestPoint_Pad_D1.0mm"
+		(property "Footprint" "TestPoint:TestPoint_THTPad_D1.0mm_Drill0.5mm"
 			(at 213.36 92.075 0)
 			(effects
@@
 			)
 		)
-		(property "Footprint" "TestPoint:TestPoint_Pad_D1.0mm"
+		(property "Footprint" "TestPoint:TestPoint_THTPad_D1.0mm_Drill0.5mm"
 			(at 151.13 89.535 0)
 			(effects
