File: Hardware/PUTM_EV_Frontbox.kicad_sch (KiCad schematic)
At the start: 4 parts

Commit message: Changes in CAN section
Other:
- sheet CAN bus ports: added GND_CAN_ISO, STBY_CAN_1, STBY_CAN_2; removed none
- sheet Connector ports: added GND_CAN_ISO; removed none
- sheet MCU ports: added STBY_CAN_1, STBY_CAN_2; removed none
- note added: "Isolated"

Commit message: Changes in schematic, separated CAN buses, added XIAO Sense S3 DevBoard
Parts:
- removed H1, H2, H3, H4: MountingHole_Pad, MountingHole:MountingHole_3.2mm_M3_Pad_Via, symbol Mechanical:MountingHole_Pad
Other:
- sheet CAN bus ports: added GND_CAN_ISO1, GND_CAN_ISO2, {CAN1_MCU}, {CAN1}, {CAN2_MCU}, {CAN2}; removed GND_CAN_ISO, {CAN_MCU}, {CAN}
- sheet Connector ports: added GND_CAN_ISO1, GND_CAN_ISO2, UART_RX, UART_TX, XIAO_GPIO, {CAN1}, {CAN2}; removed GND_CAN_ISO, {CAN}
- sheet MCU ports: added UART_RX, UART_TX, XIAO_GPIO, {CAN1_MCU}, {CAN2_MCU}; removed {CAN_MCU}

Commit message: Initial routing (Piotruś proszę nie bij że brzydko)
Other:
- sheet Connector ports: added UART_RX_PROG, UART_TX_PROG; removed none
- sheet MCU ports: added UART_RX_PROG, UART_TX_PROG; removed none
Changed lines of the file:
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@@
+	(wire
+		(pts
+			(xy 69.85 200.66) (xy 190.5 200.66)
+		)
+		(stroke
+			(width 0)
+			(type default)
+		)
+	)
 	(wire
 		(pts
@@
 		(pts
 			(xy 148.59 97.79) (xy 190.5 97.79)
+		)
+		(stroke
+			(width 0)
+			(type default)
+		)
+	)
+	(wire
+		(pts
+			(xy 69.85 196.85) (xy 190.5 196.85)
 		)
 		(stroke
@@
 			)
 		)
+		(pin "UART_RX_PROG" input
+			(at 69.85 196.85 0)
+			(effects
+				(font
+					(size 1.27 1.27)
+				)
+				(justify right)
+			)
+		)
+		(pin "UART_TX_PROG" input
+			(at 69.85 200.66 0)
+			(effects
+				(font
+					(size 1.27 1.27)
+				)
+				(justify right)
+			)
+		)
 		(instances
 			(project "PUTM_EV_Frontbox"
@@
 			)
 		)
+		(pin "UART_RX_PROG" input
+			(at 190.5 196.85 180)
+			(effects
+				(font
+					(size 1.27 1.27)
+				)
+				(justify left)
+			)
+		)
+		(pin "UART_TX_PROG" input
+			(at 190.5 200.66 180)
+			(effects
+				(font
+					(size 1.27 1.27)
+				)
+				(justify left)
+			)
+		)

Commit message: Changes in CAN section
Other:
- company: Author: -> Author: ${AUTHORS}
- title: (none) -> FrontBox
Changed lines of the file:
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@@
 	(paper "A3")
 	(title_block
+		(title "FrontBox")
 		(rev "${REVISION}")
-		(company "Author:")
-		(comment 1 "Reviewer:")
+		(company "Author: ${AUTHORS}")
+		(comment 1 "Reviewer: ${REVIEVER}")
 	)
 	(rectangle

Commit message: Added Tensionmeters initial version
Other:
- added sheet Tensionmeter (tensionmeter.kicad_sch)
- sheet Connector ports: added Tens_Out1+, Tens_Out1-, Tens_Out2+, Tens_Out2-; removed none
- sheet MCU ports: added Tens1, Tens2; removed none
Changed lines of the file:
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@@
 	(text "Clock\n"
 		(exclude_from_sim no)
-		(at 158.75 215.9 0)
+		(at 154.94 205.74 0)
 		(effects
 			(font
@@
 	(wire
 		(pts
-			(xy 182.88 209.55) (xy 182.88 223.52)
+			(xy 179.07 209.55) (xy 179.07 213.36)
 		)
 		(stroke
@@
 	(wire
 		(pts
-			(xy 190.5 209.55) (xy 182.88 209.55)
+			(xy 190.5 209.55) (xy 179.07 209.55)
 		)
 		(stroke
@@
 	(wire
 		(pts
-			(xy 171.45 223.52) (xy 182.88 223.52)
+			(xy 167.64 213.36) (xy 179.07 213.36)
 		)
 		(stroke
@@
 		)
 	)
+	(wire
+		(pts
+			(xy 69.85 214.63) (xy 119.38 214.63)
+		)
+		(stroke
+			(width 0)
+			(type default)
+		)
+	)
 	(bus
 		(pts
@@
 	(wire
 		(pts
+			(xy 138.43 222.25) (xy 190.5 222.25)
+		)
+		(stroke
+			(width 0)
+			(type default)
+		)
+	)
+	(wire
+		(pts
 			(xy 69.85 125.73) (xy 118.11 125.73)
 		)
@@
 		)
 	)
+	(wire
+		(pts
+			(xy 69.85 227.33) (xy 119.38 227.33)
+		)
+		(stroke
+			(width 0)
+			(type default)
+		)
+	)
 	(bus
 		(pts
@@
 	(wire
 		(pts
+			(xy 138.43 228.6) (xy 190.5 228.6)
+		)
+		(stroke
+			(width 0)
+			(type default)
+		)
+	)
+	(wire
+		(pts
 			(xy 148.59 101.6) (xy 190.5 101.6)
 		)
@@
 	(wire
 		(pts
+			(xy 69.85 217.17) (xy 119.38 217.17)
+		)
+		(stroke
+			(width 0)
+			(type default)
+		)
+	)
+	(wire
+		(pts
 			(xy 69.85 196.85) (xy 190.5 196.85)
+		)
+		(stroke
+			(width 0)
+			(type default)
+		)
+	)
+	(wire
+		(pts
+			(xy 69.85 223.52) (xy 119.38 223.52)
 		)
 		(stroke
@@
 	)
 	(label "HSE_IN"
-		(at 182.88 223.52 180)
+		(at 179.07 213.36 180)
 		(effects
 			(font
@@
 	(sheet
 		(at 26.67 71.12)
-		(size 43.18 134.62)
+		(size 43.18 167.64)
 		(exclude_from_sim no)
 		(in_bom yes)
@@
 		)
 		(property "Sheetfile" "Connector.kicad_sch"
-			(at 26.67 206.3246 0)
+			(at 26.67 239.3446 0)
 			(effects
 				(font
@@
 		(pin "UART_TX_PROG" input
 			(at 69.85 200.66 0)
+			(effects
+				(font
+					(size 1.27 1.27)
+				)
+				(justify right)
+			)
+		)
+		(pin "Tens_Out1+" output
+			(at 69.85 214.63 0)
+			(effects
+				(font
+					(size 1.27 1.27)
+				)
+				(justify right)
+			)
+		)
+		(pin "Tens_Out1-" output
+			(at 69.85 217.17 0)
+			(effects
+				(font
+					(size 1.27 1.27)
+				)
+				(justify right)
+			)
+		)
+		(pin "Tens_Out2+" output
+			(at 69.85 223.52 0)
+			(effects
+				(font
+					(size 1.27 1.27)
+				)
+				(justify right)
+			)
+		)
+		(pin "Tens_Out2-" output
+			(at 69.85 227.33 0)
 			(effects
 				(font
@@
 	)
 	(sheet
-		(at 153.67 220.98)
+		(at 149.86 210.82)
 		(size 17.78 5.08)
 		(exclude_from_sim no)
@@
 		)
 		(property "Sheetname" "Oscillator"
-			(at 153.67 220.2684 0)
+			(at 149.86 210.1084 0)
 			(effects
 				(font
@@
 		)
 		(property "Sheetfile" "oscillator.kicad_sch"
-			(at 153.67 226.6446 0)
+			(at 149.86 216.4846 0)
 			(effects
 				(font
@@
 		)
 		(pin "HSE_IN" output
-			(at 171.45 223.52 0)
+			(at 167.64 213.36 0)
 			(effects
 				(font
@@
 	)
 	(sheet
+		(at 119.38 210.82)
+		(size 19.05 22.86)
+		(exclude_from_sim no)
+		(in_bom yes)
+		(on_board yes)
+		(dnp no)
+		(fields_autoplaced yes)
+		(stroke
+			(width 0.1524)
+			(type solid)
+		)
+		(fill
+			(color 0 0 0 0.0000)
+		)
+		(property "Sheetname" "Tensionmeter"
+			(at 119.38 210.1084 0)
+			(effects
+				(font
+					(size 1.27 1.27)
+				)
+				(justify left bottom)
+			)
+		)
+		(property "Sheetfile" "tensionmeter.kicad_sch"
+			(at 119.38 234.2646 0)
+			(effects
+				(font
+					(size 1.27 1.27)
+				)
+				(justify left top)
+			)
+		)
+		(pin "OUT1+" input
+			(at 119.38 214.63 180)
+			(effects
+				(font
+					(size 1.27 1.27)
+				)
+				(justify left)
+			)
+		)
+		(pin "OUT1-" input
+			(at 119.38 217.17 180)
+			(effects
+				(font
+					(size 1.27 1.27)
+				)
+				(justify left)
+			)
+		)
+		(pin "OUT2+" input
+			(at 119.38 223.52 180)
+			(effects
+				(font
+					(size 1.27 1.27)
+				)
+				(justify left)
+			)
+		)
+		(pin "OUT2-" input
+			(at 119.38 227.33 180)
+			(effects
+				(font
+					(size 1.27 1.27)
+				)
+				(justify left)
+			)
+		)
+		(pin "Tens1" output
+			(at 138.43 222.25 0)
+			(effects
+				(font
+					(size 1.27 1.27)
+				)
+				(justify right)
+			)
+		)
+		(pin "Tens2" output
+			(at 138.43 228.6 0)
+			(effects
+				(font
+					(size 1.27 1.27)
+				)
+				(justify right)
+			)
+		)
+		(instances
+			(project "PUTM_EV_Frontbox"
+				(path "/b652b05a-4e3d-4ad1-b032-18886abe7d45"
+					(page "12")
+				)
+			)
+		)
+	)
+	(sheet
 		(at 118.11 93.98)
 		(size 30.48 12.7)
@@
 	(sheet
 		(at 190.5 69.85)
-		(size 62.23 147.32)
+		(size 62.23 167.64)
 		(exclude_from_sim no)
 		(in_bom yes)
@@
 		)
 		(property "Sheetfile" "STM.kicad_sch"
-			(at 190.5 217.7546 0)
+			(at 190.5 238.0746 0)
 			(effects
 				(font
@@
 			(effects
 				(font
+					(size 1.27 1.27)
+				)
+				(justify left)
+			)
+		)
+		(pin "Tens1" input
+			(at 190.5 222.25 180)
+			(effects
+				(font
+					(size 1.27 1.27)
+				)
+				(justify left)
+			)
+		)
+		(pin "Tens2" input
+			(at 190.5 228.6 180)
+			(effects
+				(font
