File: Hardware/STM.kicad_sch (KiCad schematic)
At the start: 26 parts, among them U5 LM4040C33FTA, U6 STM32G484RETx

Commit message: Added Tensionmeters initial version
Connections:
- net Tens1: now reaches U6.12 (PA0)
- net Tens2: now reaches U6.13 (PA1)
- no-connect marks 16 -> 14
Changed lines of the file:
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@@
 	)
 	(no_connect
-		(at 157.48 60.96)
-	)
-	(no_connect
 		(at 157.48 106.68)
 	)
@@
 	)
 	(no_connect
-		(at 157.48 58.42)
-	)
-	(no_connect
 		(at 157.48 104.14)
 	)
@@
 	(wire
 		(pts
+			(xy 161.29 58.42) (xy 157.48 58.42)
+		)
+		(stroke
+			(width 0)
+			(type default)
+		)
+	)
+	(wire
+		(pts
 			(xy 86.36 58.42) (xy 121.92 58.42)
 		)
@@
 	(wire
 		(pts
+			(xy 161.29 60.96) (xy 157.48 60.96)
+		)
+		(stroke
+			(width 0)
+			(type default)
+		)
+	)
+	(wire
+		(pts
 			(xy 186.69 39.37) (xy 173.99 39.37)
 		)
@@
 		)
 	)
+	(hierarchical_label "Tens2"
+		(shape input)
+		(at 161.29 60.96 0)
+		(effects
+			(font
+				(size 1.27 1.27)
+			)
+			(justify left)
+		)
+	)
 	(hierarchical_label "{CAN1_MCU}"
 		(shape bidirectional)
@@
 		)
 	)
+	(hierarchical_label "Tens1"
+		(shape input)
+		(at 161.29 58.42 0)
+		(effects
+			(font
+				(size 1.27 1.27)
+			)
+			(justify left)
+		)
+	)
 	(hierarchical_label "DAC1_REF"
 		(shape output)
@@
 		)
 		(pin "12"
+			(alternate "ADC1_IN1")
 		)
 		(pin "19"
@@
 		)
 		(pin "13"
+			(alternate "ADC1_IN2")
 		)
 		(pin "25"
@@
 					(unit 1)
 				)
-			)
-		)
-	)
-	(symbol
-		(lib_id "power:PWR_FLAG")
-		(at 247.65 27.94 270)
-		(unit 1)
-		(exclude_from_sim no)
-		(in_bom yes)
-		(on_board yes)
-		(dnp no)
-		(fields_autoplaced yes)
-		(property "Reference" "#FLG013"
-			(at 249.555 27.94 0)
-			(effects
-				(font
-					(size 1.27 1.27)
-				)
-				(hide yes)
-			)
-		)
-		(property "Value" "PWR_FLAG"
-			(at 251.46 27.9399 90)
-			(effects
-				(font
-					(size 1.27 1.27)
-				)
-				(justify left)
-			)
-		)
-		(property "Footprint" ""
-			(at 247.65 27.94 0)
-			(effects
-				(font
-					(size 1.27 1.27)
-				)
-				(hide yes)
-			)
-		)
-		(property "Datasheet" "~"
-			(at 247.65 27.94 0)
-			(effects
-				(font
-					(size 1.27 1.27)
-				)
-				(hide yes)
-			)
-		)
-		(property "Description" ""
-			(at 247.65 27.94 0)
-			(effects
-				(font
-					(size 1.27 1.27)
-				)
-				(hide yes)
-			)
-		)
-		(pin "1"
-		)
-		(instances
-			(project "PUTM_EV_Frontbox"
-				(path "/b652b05a-4e3d-4ad1-b032-18886abe7d45/bb657190-4781-414f-856e-04fa26549ae4"
-					(reference "#FLG013")
-					(unit 1)
-				)
