File: Hardware/Connector.kicad_sch (KiCad schematic)
At the start: 14 parts, among them J1 XIAO ESP32S3 Sense, J2 Conn_02x16_Counter_Clockwise, J3 FTSH-107-01-L-D-K

Commit message: First iteration to send
Parts:
- F6: Mouser Part Number . -> 603-SMD0603B010TF
- J1: now not fitted
Changed lines of the file:
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@@
 			)
 		)
-		(property "Mouser Part Number" "."
+		(property "Mouser Part Number" "603-SMD0603B010TF"
 			(at 144.78 72.39 0)
 			(effects
@@
 					(size 1.27 1.27)
 				)
+				(hide yes)
 			)
 		)
@@
 		(in_bom yes)
 		(on_board yes)
-		(dnp no)
+		(dnp yes)
 		(property "Reference" "J1"
 			(at 251.46 48.2599 0)
